File: hardware/core_pcb/cems_core.kicad_sch (KiCad schematic)
At the start: 0 parts

Commit message: CORE PCB rev 0.2: I/O node section on the same board
Three new sheets: field digital I/O with the hardware output gate (ISO2H823V2.5,
ISO808A-1, ISO1I813T), field power / pump / relay coils / USB-C, and the isolated
analog (AD4112) and temperature (ADS124S08) islands. Project symbols for the six
I/O chips missing from KiCad. SPI4 nets renamed: the bus is shared with the I/O chips.
423 parts, netlist check passes. CORE_PCB.md: pin map, connectors, BOM, section 14.

Co-Authored-By: Claude Opus 5.5 <noreply@anthropic.com>
Claude-Session: https://claude.ai/code/session_014onnq3eRiDkqdAB6fKiRDW
Other:
- added sheet Analog inputs and temperatures (io_ana.kicad_sch)
- added sheet Field digital I/O (io_dig.kicad_sch)
- added sheet Field power, pump, relays, USB (io_pwr.kicad_sch)
Changed lines of the file:
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@@
   (title_block
     (title "CEMS core board")
-    (date "2026-10-25")
-    (rev "0.1")
+    (date "2026-10-31")
+    (rev "0.2")
     (company "EnviroDevelo")
     (comment 1 "Generated from hardware/core_pcb/tools/design.py; do not edit by hand")
@@
       )
     )
+  )
+  (sheet (at 20 85) (size 45 25) (fields_autoplaced)
+    (stroke (width 0.0))
+    (fill (color 0 0 0 0))
+    (property "Sheetname" "Field digital I/O" (id 0) (at 20 84.3 0)
+      (effects (font (size 1.27 1.27)) (justify left bottom))
+    )
+    (property "Sheetfile" "io_dig.kicad_sch" (id 1) (at 20 110.6 0)
+      (effects (font (size 1.27 1.27)) (justify left top))
+    )
+    (instances
+      (project "cems_core"
+        (path "/4503b035-ec93-58ad-a08a-2d339f99cb7b" (page "7"))
+      )
+    )
+  )
+  (sheet (at 72 85) (size 45 25) (fields_autoplaced)
+    (stroke (width 0.0))
+    (fill (color 0 0 0 0))
+    (property "Sheetname" "Field power, pump, relays, USB" (id 0) (at 72 84.3 0)
+      (effects (font (size 1.27 1.27)) (justify left bottom))
+    )
+    (property "Sheetfile" "io_pwr.kicad_sch" (id 1) (at 72 110.6 0)
+      (effects (font (size 1.27 1.27)) (justify left top))
+    )
+    (instances
+      (project "cems_core"
+        (path "/4503b035-ec93-58ad-a08a-2d339f99cb7b" (page "8"))
+      )
+    )
+  )
+  (sheet (at 124 85) (size 45 25) (fields_autoplaced)
+    (stroke (width 0.0))
+    (fill (color 0 0 0 0))
+    (property "Sheetname" "Analog inputs and temperatures" (id 0) (at 124 84.3 0)
+      (effects (font (size 1.27 1.27)) (justify left bottom))
+    )
+    (property "Sheetfile" "io_ana.kicad_sch" (id 1) (at 124 110.6 0)
+      (effects (font (size 1.27 1.27)) (justify left top))
+    )
+    (instances
+      (project "cems_core"
+        (path "/4503b035-ec93-58ad-a08a-2d339f99cb7b" (page "9"))
+      )
+    )
