File: hardware/core_pcb/eth_client.kicad_sch (KiCad schematic)
At the start: 27 parts, among them J2 CLIENT, U4 LAN8742A-CZ, U5 TPD4E05U06, Y3 25MHz

Commit message: Core PCB: save datasheets and clear the datasheet checks
Add hardware/datasheets with the six datasheets Gary supplied and an index.
Apply what they show: TPS54360B with 22 uH and compensation from its
datasheet, LAN8742A crystal caps 33 pF, W5500 reserved pins 38-42 left open
and its reference crystal circuit (1M, 0R), FRAM and choke checks cleared.

Co-Authored-By: Claude Opus 5.5 (1M context) <noreply@anthropic.com>
Claude-Session: https://claude.ai/code/session_014onnq3eRiDkqdAB6fKiRDW
Parts:
- C46, C47: value 15p -> 33p; MPN 15p -> 33p
Other:
- note added: "Notes U4: straps: MODE[2:0] internal pull-ups = all capable; PHYAD0 internal pull-down = address 0; nINTSEL pulled low (R33) = pin 14 is REFCLKO, 50 MHz to the MCU; REGOFF internal pull-down = regulator on C41: at pin 1 C42: at pin 19 C43: VDDIO C44: VDDCR, with C45 Y3: CL 20 pF, +/-50 ppm total (LAN8742A datasheet) C46: for CL 20 pF with about 4 pF stray"
- note removed: "Notes U4: straps: MODE[2:0] internal pull-ups = all capable; PHYAD0 internal pull-down = address 0; nINTSEL pulled low (R33) = pin 14 is REFCLKO, 50 MHz to the MCU; REGOFF internal pull-down = regulator on C41: at pin 1 C42: at pin 19 C43: VDDIO C44: VDDCR, with C45 Y3: +/-50 ppm or better C46: CHECK for the crystal's CL"
Changed lines of the file:
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@@
   (no_connect (at 30.48 127.0))
   (no_connect (at 127.0 119.38))
-  (text "Notes\nU4: straps: MODE[2:0] internal pull-ups = all capable; PHYAD0 internal pull-down = address 0; nINTSEL pulled low (R33) = pin 14 is REFCLKO, 50 MHz to the MCU; REGOFF internal pull-down = regulator on\nC41: at pin 1\nC42: at pin 19\nC43: VDDIO\nC44: VDDCR, with C45\nY3: +/-50 ppm or better\nC46: CHECK for the crystal's CL"
+  (text "Notes\nU4: straps: MODE[2:0] internal pull-ups = all capable; PHYAD0 internal pull-down = address 0; nINTSEL pulled low (R33) = pin 14 is REFCLKO, 50 MHz to the MCU; REGOFF internal pull-down = regulator on\nC41: at pin 1\nC42: at pin 19\nC43: VDDIO\nC44: VDDCR, with C45\nY3: CL 20 pF, +/-50 ppm total (LAN8742A datasheet)\nC46: for CL 20 pF with about 4 pF stray"
     (at 15.24 226.06 0)
     (effects (font (size 1.0 1.0)) (justify left top))
@@
       (effects (font (size 1.27 1.27)))
     )
-    (property "Value" "15p" (id 1) (at 231.14000000000001 50.8 0)
+    (property "Value" "33p" (id 1) (at 231.14000000000001 50.8 0)
       (effects (font (size 1.27 1.27)))
     )
@@
       (effects (font (size 1.27 1.27)) hide)
     )
-    (property "MPN" "15p" (id 4) (at 231.14000000000001 35.56 0)
+    (property "MPN" "33p" (id 4) (at 231.14000000000001 35.56 0)
       (effects (font (size 1.27 1.27)) hide)
     )
@@
       (effects (font (size 1.27 1.27)))
     )
-    (property "Value" "15p" (id 1) (at 243.84 50.8 0)
+    (property "Value" "33p" (id 1) (at 243.84 50.8 0)
       (effects (font (size 1.27 1.27)))
     )
@@
       (effects (font (size 1.27 1.27)) hide)
     )
-    (property "MPN" "15p" (id 4) (at 243.84 35.56 0)
-      (effects (font (size 1.27 1.27)) hide)
-    )
+    (property "MPN" "33p" (id 4) (at 243.84 35.56 0)
+      (effects (font (size 1.27 1.27)) hide)
+    )

Commit message: Core PCB: RMII series terminations and the any-switch / 100 m design rules
33R source series resistors on TX_EN/TXD0/TXD1 (at the MCU) and
CRS_DV/RXD0/RXD1 (at the PHY), as on ST's DK. CORE_PCB.md 7 records what
the 100 m / any-switch requirement (Gary, 30 Oct) rests on: PHY crystal and
REFCLKO, MODE 111 auto-negotiation (never forced), PHY reset under firmware
control, reference line termination and differential-pair routing.

Co-Authored-By: Claude Opus 5.5 <noreply@anthropic.com>
Claude-Session: https://claude.ai/code/session_014onnq3eRiDkqdAB6fKiRDW
Parts:
- added R41, R42, R43, R44, R45, R46: 33R, Resistor_SMD:R_0603_1608Metric, symbol Device:R
Connections:
- net ETH_CRS_DV: now also R44.2; no longer U4.11 (CRS_DV/MODE2)
- net ETH_RXD0: now also R45.2; no longer U4.8 (RXD0/MODE0)
- net ETH_RXD1: now also R46.2; no longer U4.7 (RXD1/MODE1)
- net ETH_TXD0: now also R42.2
- net ETH_TXD1: now also R43.2
- net ETH_TX_EN: now also R41.2
- new net ETH_TXD0_MCU: R42.1
- new net ETH_TXD1_MCU: R43.1
- new net ETH_TX_EN_MCU: R41.1
- new net PHY_CRS_DV: R44.1, U4.11 (CRS_DV/MODE2)
- new net PHY_RXD0: R45.1, U4.8 (RXD0/MODE0)
- new net PHY_RXD1: R46.1, U4.7 (RXD1/MODE1)
Other:
- note added: "Notes U4: straps: MODE[2:0] internal pull-ups = all capable; PHYAD0 internal pull-down = address 0; nINTSEL pulled low (R33) = pin 14 is REFCLKO, 50 MHz to the MCU; REGOFF internal pull-down = regulator on C41: at pin 1 C42: at pin 19 C43: VDDIO C44: VDDCR, with C45 Y3: CL 20 pF, +/-50 ppm total (LAN8742A datasheet) C46: for CL 20 pF with about 4 pF stray R31: series, at the PHY R41: series, at t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"
- note added: "R43: series, at the MCU R44: series, at the PHY R45: series, at the PHY R46: series, at the PHY R33: strap nINTSEL = 0 (REFCLKO mode) R34: PHY runs if the firmware leaves PD11 as input U5: flow-through: route each line across pins 1/10, 2/9, 4/7, 5/6 J2: client network R39: LED1 = link/activity, active high (REGOFF strap low) R40: LED2 = speed, active high (nINTSEL strap low)"
- note removed: "Notes U4: straps: MODE[2:0] internal pull-ups = all capable; PHYAD0 internal pull-down = address 0; nINTSEL pulled low (R33) = pin 14 is REFCLKO, 50 MHz to the MCU; REGOFF internal pull-down = regulator on C41: at pin 1 C42: at pin 19 C43: VDDIO C44: VDDCR, with C45 Y3: CL 20 pF, +/-50 ppm total (LAN8742A datasheet) C46: for CL 20 pF with about 4 pF stray"
- note removed: "R31: series, at the PHY R33: strap nINTSEL = 0 (REFCLKO mode) R34: PHY runs if the firmware leaves PD11 as input U5: flow-through: route each line across pins 1/10, 2/9, 4/7, 5/6 J2: client network R39: LED1 = link/activity, active high (REGOFF strap low) R40: LED2 = speed, active high (nINTSEL strap low)"
- moved on the sheet: C48, C49, FB3, J2, R32, R33, R34, R35, R36, R37, R38, R39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
