File: hardware/core_pcb/io_ana.kicad_sch (KiCad schematic)
At the start: 89 parts, among them J19 TEMP1, J20 TEMP2, J21 TEMP3, J22 AI 1-2, J23 AI 3-4, J24 AI 5-6, J25 SENSORS, U28 ISOW7741, U29 74LVC1G04, U30 ADS124S08, U31 ISOW7741, U32 74LVC1G04, U33 ITX2424SA, U34 AD4112, U35 L78L05, U36 LM317L, U37 REF5010, U38 LT3045

Commit message: CORE PCB: I/O chip pinouts checked against datasheets; gate latch, ODIS polarity
Pin tables of AD4112, ADS124S08, ISO2H823V2.5, ISO1I813T, ISO808A-1, ISO7741 and
ISOW7741 compared with the datasheets: all match. Fixes from the check: ISO2H823 /ODIS
is active low (takes GATE directly); OLADJ fitted 12.1k; CLKADJ 10k 0.1 %; ROSC 22.1k;
ISOW7741 EN/FLT pulled to 3.3 V; MAX6369 WDO only pulses, so a 74LVC1G175 latches a
trip until GATE_EN is re-armed. hardware/datasheets/IO_CHIPS_DATASHEET_CHECK.md holds the
extracts and the AD4112 register facts for the driver.

Co-Authored-By: Claude Opus 5.5 <noreply@anthropic.com>
Claude-Session: https://claude.ai/code/session_014onnq3eRiDkqdAB6fKiRDW
Connections:
- net +3V3: now also R164.1, R176.1
- net +5V: no longer R164.1, R176.1
Other:
- note added: "J21: T5 +/-, T6 +/-, RTD return U31: VSEL to VISOOUT = 5 V out (110 mA) R176: EN/FLT high (VIO level) enables the DC/DC; reads low on a fault U33: loop power 6 x 22 mA + level + mass-flow supply, about 4 W U34: internal oscillator and 2.5 V reference. VIN0/1: 4-20 mA ch 5/6 on shunts; VIN2 level; VIN3 mass flow; VIN4 10 V monitor; VIN5 5 V monitor. Pinout checked (31 Oct); CHECK the exposed pad s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"
- note added: "J24: per channel: 24 V loop, IN, 0 V (2-wire or 4-wire transmitters) U35: level sensor 5 V, internal current limit R180: defined level when unplugged U36: 13 V pre-regulator, about 0.5 W: copper on the VO pins R182: 1.25 x (1 + 2260/240) = 13.0 V U38: SET driven by the REF5010 (no RSET). CHECK PGFB tie when PG is unused R183: about 50 mA current limit R184: 10 V monitor for ratiometric correction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"
- note added: "Notes U28: VSEL to GND2 = 3.3 V out (140 mA) R164: EN/FLT high (VIO level) enables the DC/DC; reads low on a fault U30: pinout checked (SBAS660, 31 Oct). Internal 4.096 MHz clock (CLK to DGND), START low (conversions by command), DOUT/DRDY on one pin C145: REFOUT to REFCOM R166: RTD reference resistor, 10 ppm/K C147: CHECK AINCOM and the TC bias against the io-node schematic C148: differential fi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"
- note removed: "J21: T5 +/-, T6 +/-, RTD return U31: VSEL high = 5 V out. CHECK U33: loop power 6 x 22 mA + level + mass-flow supply, about 4 W U34: internal oscillator and 2.5 V reference. VIN0/1: 4-20 mA ch 5/6 on shunts; VIN2 level; VIN3 mass flow; VIN4 10 V monitor; VIN5 5 V monitor. CHECK pinout and exposed pad size R178: 4-20 mA shunt -> 1-5 V R179: 4-20 mA shunt -> 1-5 V F16: loop supply limit J22: per ch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"
- note removed: "Notes U28: VSEL low = 3.3 V out. CHECK U30: internal clock (CLK low), START low (conversions by command), DOUT/DRDY on one pin. CHECK pinout C145: REFOUT to REFCOM R166: RTD reference resistor, 10 ppm/K C147: CHECK AINCOM and the TC bias against the io-node schematic C148: differential filter R167: open-TC bias R173: RTD return to the reference resistor J19: T1 +/-, T2 +/-, RTD return J20: T3 +/-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"
- note removed: "U35: level sensor 5 V, internal current limit R180: defined level when unplugged U36: 13 V pre-regulator, about 0.5 W: copper on the VO pins R182: 1.25 x (1 + 2260/240) = 13.0 V U38: SET driven by the REF5010 (no RSET). CHECK PGFB tie when PG is unused R183: about 50 mA current limit R184: 10 V monitor for ratiometric correction J25: level (DFRobot SEN0205): 5 V, SIG, 0 V; mass flow (AWM5104VN): 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"
- moved on the sheet: R176
Changed lines of the file:
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@@
   (no_connect (at 264.16 190.5))
   (no_connect (at 342.90000000000003 182.88000000000002))
-  (text "Notes\nU28: VSEL low = 3.3 V out. CHECK\nU30: internal clock (CLK low), START low (conversions by command), DOUT/DRDY on one pin. CHECK pinout\nC145: REFOUT to REFCOM\nR166: RTD reference resistor, 10 ppm/K\nC147: CHECK AINCOM and the TC bias against the io-node schematic\nC148: differential filter\nR167: open-TC bias\nR173: RTD return to the reference resistor\nJ19: T1 +/-, T2 +/-, RTD return\nJ20: T3 +/-, T4 +/-, RTD return"
+  (text "Notes\nU28: VSEL to GND2 = 3.3 V out (140 mA)\nR164: EN/FLT high (VIO level) enables the DC/DC; reads low on a fault\nU30: pinout checked (SBAS660, 31 Oct). Internal 4.096 MHz clock (CLK to DGND), START low (conversions by command), DOUT/DRDY on one pin\nC145: REFOUT to REFCOM\nR166: RTD reference resistor, 10 ppm/K\nC147: CHECK AINCOM and the TC bias against the io-node schematic\nC148: differential filter\nR167: open-TC bias\nR173: RTD return to the reference resistor\nJ19: T1 +/-, T2 +/-, RTD return\nJ20: T3 +/-, T4 +/-, RTD return"
     (at 15.24 347.98 0)
     (effects (font (size 1.0 1.0)) (justify left top))
   )
-  (text "\nJ21: T5 +/-, T6 +/-, RTD return\nU31: VSEL high = 5 V out. CHECK\nU33: loop power 6 x 22 mA + level + mass-flow supply, about 4 W\nU34: internal oscillator and 2.5 V reference. VIN0/1: 4-20 mA ch 5/6 on shunts; VIN2 level; VIN3 mass flow; VIN4 10 V monitor; VIN5 5 V monitor. CHECK pinout and exposed pad size\nR178: 4-20 mA shunt -> 1-5 V\nR179: 4-20 mA shunt -> 1-5 V\nF16: loop supply limit\nJ22: per channel: 24 V loop, IN, 0 V (2-wire or 4-wire transmitters)\nJ23: per channel: 24 V loop, IN, 0 V (2-wire or 4-wire transmitters)\nJ24: per channel: 24 V loop, IN, 0 V (2-wire or 4-wire transmitters)"
+  (text "\nJ21: T5 +/-, T6 +/-, RTD return\nU31: VSEL to VISOOUT = 5 V out (110 mA)\nR176: EN/FLT high (VIO level) enables the DC/DC; reads low on a fault\nU33: loop power 6 x 22 mA + level + mass-flow supply, about 4 W\nU34: internal oscillator and 2.5 V reference. VIN0/1: 4-20 mA ch 5/6 on shunts; VIN2 level; VIN3 mass flow; VIN4 10 V monitor; VIN5 5 V monitor. Pinout checked (31 Oct); CHECK the exposed pad size against\n    the CP-40 drawing\nR178: 4-20 mA shunt -> 1-5 V\nR179: 4-20 mA shunt -> 1-5 V\nF16: loop supply limit\nJ22: per channel: 24 V loop, IN, 0 V (2-wire or 4-wire transmitters)\nJ23: per channel: 24 V loop, IN, 0 V (2-wire or 4-wire transmitters)"
     (at 203.2 347.98 0)
     (effects (font (size 1.0 1.0)) (justify left top))
   )
-  (text "\nU35: level sensor 5 V, internal current limit\nR180: defined level when unplugged\nU36: 13 V pre-regulator, about 0.5 W: copper on the VO pins\nR182: 1.25 x (1 + 2260/240) = 13.0 V\nU38: SET driven by the REF5010 (no RSET). CHECK PGFB tie when PG is unused\nR183: about 50 mA current limit\nR184: 10 V monitor for ratiometric correction\nJ25: level (DFRobot SEN0205): 5 V, SIG, 0 V; mass flow (AWM5104VN): +10 V, OUT, 0 V"
+  (text "\nJ24: per channel: 24 V loop, IN, 0 V (2-wire or 4-wire transmitters)\nU35: level sensor 5 V, internal current limit\nR180: defined level when unplugged\nU36: 13 V pre-regulator, about 0.5 W: copper on the VO pins\nR182: 1.25 x (1 + 2260/240) = 13.0 V\nU38: SET driven by the REF5010 (no RSET). CHECK PGFB tie when PG is unused\nR183: about 50 mA current limit\nR184: 10 V monitor for ratiometric correction\nJ25: level (DFRobot SEN0205): 5 V, SIG, 0 V; mass flow (AWM5104VN): +10 V, OUT, 0 V"
     (at 391.16 347.98 0)
     (effects (font (size 1.0 1.0)) (justify left top))
@@
     (effects (font (size 1.27 1.27)) (justify right))
   )
-  (label "AI_ENFLT" (at 185.42000000000002 105.41 270)
+  (label "AI_ENFLT" (at 185.42000000000002 107.95 270)
     (effects (font (size 1.27 1.27)) (justify right))
   )
@@
     )
   )
-  (global_label "+5V" (shape passive) (at 147.32 29.210000000000004 90) (fields_autoplaced)
+  (global_label "+3V3" (shape passive) (at 147.32 29.210000000000004 90) (fields_autoplaced)
     (effects (font (size 1.27 1.27)) (justify left))
     (property "Intersheetrefs" "${INTERSHEET_REFS}" (id 0) (at 147.32 29.210000000000004 90)
@@
     )
   )
-  (global_label "+5V" (shape passive) (at 185.42000000000002 97.78999999999999 90) (fields_autoplaced)
-    (effects (font (size 1.27 1.27)) (justify left))
-    (property "Intersheetrefs" "${INTERSHEET_REFS}" (id 0) (at 185.42000000000002 97.78999999999999 90)
+  (global_label "+3V3" (shape passive) (at 185.42000000000002 100.33 90) (fields_autoplaced)
+    (effects (font (size 1.27 1.27)) (justify left))
+    (property "Intersheetrefs" "${INTERSHEET_REFS}" (id 0) (at 185.42000000000002 100.33 90)
       (effects (font (size 1.27 1.27)) (justify left) hide)
     )
@@
     )
   )
-  (symbol (lib_id "Device:R") (at 185.42000000000002 101.6 0) (unit 1)
-    (in_bom yes) (on_board yes) (dnp no)
-    (property "Reference" "R176" (id 0) (at 185.42000000000002 86.36 0)
-      (effects (font (size 1.27 1.27)))
-    )
-    (property "Value" "10k" (id 1) (at 185.42000000000002 119.38 0)
-      (effects (font (size 1.27 1.27)))
-    )
-    (property "Footprint" "Resistor_SMD:R_0603_1608Metric" (id 2) (at 185.42000000000002 101.6 0)
-      (effects (font (size 1.27 1.27)) hide)
-    )
-    (property "Datasheet" "~" (id 3) (at 185.42000000000002 101.6 0)
-      (effects (font (size 1.27 1.27)) hide)
-    )
-    (property "MPN" "10k" (id 4) (at 185.42000000000002 101.6 0)
-      (effects (font (size 1.27 1.27)) hide)
-    )
+  (symbol (lib_id "Device:R") (at 185.42000000000002 104.14 0) (unit 1)
+    (in_bom yes) (on_board yes) (dnp no)
+    (property "Reference" "R176" (id 0) (at 185.42000000000002 88.9 0)
+      (effects (font (size 1.27 1.27)))
+    )
+    (property "Value" "10k" (id 1) (at 185.42000000000002 121.92 0)
+      (effects (font (size 1.27 1.27)))
+    )
+    (property "Footprint" "Resistor_SMD:R_0603_1608Metric" (id 2) (at 185.42000000000002 104.14 0)
+      (effects (font (size 1.27 1.27)) hide)
+    )
+    (property "Datasheet" "~" (id 3) (at 185.42000000000002 104.14 0)
+      (effects (font (size 1.27 1.27)) hide)
+    )
+    (property "MPN" "10k" (id 4) (at 185.42000000000002 104.14 0)
+      (effects (font (size 1.27 1.27)) hide)
+    )

Commit message: CORE PCB + breakout: make every user plug fit only its own header
Three pitch families (5.08 power/24 V outputs, 3.81 bank B, 3.5 sensors), one size per
header except the harmless temperature and 4-20 mA groups, and a coding key per header
(script-checked against every plug and shift). J13+J14 merged into one 4-way field plug;
pump power and signals on one 6-way plug (J16 gone); relays 3-way. Survival layer: 1k 1 W
pump outputs, per-channel relay PTCs + CPC1014N, 30 mA loop current limiters, TVS on the
5 V and 10 V sensor supplies. CORE_PCB.md section 15 has the mis-plug tables.

Co-Authored-By: Claude Opus 5.5 <noreply@anthropic.com>
Claude-Session: https://claude.ai/code/session_014onnq3eRiDkqdAB6fKiRDW
Parts:
- added D49: SMAJ5.0A, Diode_SMD:D_SMA, symbol Device:D_Zener
- added D50: SMAJ11A, Diode_SMD:D_SMA, symbol Device:D_Zener
- F16, F17, F18, F19, F20, F21: value 50mA -> CCR 30mA; footprint Fuse:Fuse_1206_3216Metric -> Diode_SMD:D_PowerDI-123; symbol Device:Polyfuse -> Device:D; MPN Bourns MF-NSMF005-2 (or a 30 mA current limiter) -> Diodes AL5809-30P1-7 (60 V, 30 mA)
- J19, J20, J21: footprint Connector_Phoenix_MC:PhoenixContact_MCV_1,5_5-G-3.81_1x05_P3.81mm_Vertical -> Connector_Phoenix_MC:PhoenixContact_MCV_1,5_5-G-3.5_1x05_P3.50mm_Vertical; MPN Phoenix MCV 1,5/5-G-3,81 (or Degson / Dinkle equivalent) + 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 -> Phoenix MCV 1,5/5-G-3,5 + coded, labelled plug; coding key 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
- J22, J23, J24: footprint Connector_Phoenix_MC:PhoenixContact_MCV_1,5_6-G-3.81_1x06_P3.81mm_Vertical -> Connector_Phoenix_MC:PhoenixContact_MCV_1,5_6-G-3.5_1x06_P3.50mm_Vertical; MPN Phoenix MCV 1,5/6-G-3,81 (or Degson / Dinkle equivalent) + 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 -> Phoenix MCV 1,5/6-G-3,5 + coded, labelled plug; coding key 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
- J25: footprint Connector_Phoenix_MC:PhoenixContact_MCV_1,5_6-G-3.81_1x06_P3.81mm_Vertical -> Connector_Phoenix_MC:PhoenixContact_MCV_1,5_7-G-3.5_1x07_P3.50mm_Vertical; symbol Connector_Generic:Conn_01x06 -> Connector_Generic:Conn_01x07; MPN Phoenix MCV 1,5/6-G-3,81 (or Degson / Dinkle equivalent) + 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 -> Phoenix MCV 1,5/7-G-3,5 + coded, labelled plug; coding key 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
- R178, R179: footprint Resistor_SMD:R_0805_2012Metric -> Resistor_SMD:R_1206_3216Metric; MPN 10 ppm/K thin film -> Vishay PTN1206 0.4 W, 10 ppm/K thin film
Connections:
- net +10V_FLOW: now also D50.1 (K)
- net +24V_AI: now also F16.2 (A), F17.2 (A), F18.2 (A), F19.2 (A), F20.2 (A), F21.2 (A); no longer F16.1, F17.1, F18.1, F19.1, F20.1, F21.1
- net +5V_LVL: now also D49.1 (K)
- net GND_AI: now also J25.7 (Pin_7), D49.2 (A), D50.2 (A)
- net LOOP1: now also F16.1 (K); no longer F16.2
- net LOOP2: now also F17.1 (K); no longer F17.2
- net LOOP3: now also F18.1 (K); no longer F18.2
- net LOOP4: now also F19.1 (K); no longer F19.2
- net LOOP5: now also F20.1 (K); no longer F20.2
- net LOOP6: now also F21.1 (K); no longer F21.2
Other:
- moved on the sheet: C169, C170, C171, C172, C173, C174, C175, F16, F17, F18, F19, F20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

Commit message: CORE PCB: fit-optional 4 x 4-20 mA analog outputs (AD5755-1, all DNP)
AD5755-1 on the analog island with its own ISOW7741 (CS_AO on PD3) and an ITX2405SA for
the boost converters; keyed 8-way 3.5 mm J26 (keys 2, 6, script-checked). Pin numbers from
the datasheet Table 5. Layout block plan now 2.8 mm over in io_pwr: the board is full
single-sided, see thread for the module option.

Co-Authored-By: Claude Opus 5.5 <noreply@anthropic.com>
Claude-Session: https://claude.ai/code/session_014onnq3eRiDkqdAB6fKiRDW
Parts:
- removed R164: 10k, Resistor_SMD:R_0603_1608Metric, symbol Device:R
- added C301, C303, C304, C306, C309, C326, C329: 100n, Capacitor_SMD:C_0603_1608Metric, symbol Device:C
- added C302, C305, C327: 10u, Capacitor_SMD:C_0805_2012Metric, symbol Device:C
- added C307: 10u 50V, Capacitor_SMD:C_1210_3225Metric, symbol Device:C
- added C308: 22u, Capacitor_SMD:C_1210_3225Metric, symbol Device:C
- added C310, C314, C318, C322: 4u7 50V, Capacitor_SMD:C_1210_3225Metric, symbol Device:C
- added C311, C315, C319, C323, C328: 100n 50V, Capacitor_SMD:C_0603_1608Metric, symbol Device:C
- added C312, C316, C320, C324: 10n, Capacitor_SMD:C_0603_1608Metric, symbol Device:C
- added C313, C317, C321, C325: 4n7 50V, Capacitor_SMD:C_0603_1608Metric, symbol Device:C
- added D51, D52, D53, D54: PMEG4010, Diode_SMD:D_SOD-323F, symbol Device:D_Schottky
- added D55, D56, D57, D58: SMAJ33A, Diode_SMD:D_SMA, symbol Device:D_Zener
- added J26: AO 1-4, Connector_Phoenix_MC:PhoenixContact_MCV_1,5_8-G-3.5_1x08_P3.50mm_Vertical, symbol Connector_Generic:Conn_01x08
- added L4, L5, L6, L7: 10uH, Inductor_SMD:L_Coilcraft_XAL4040-XXX, symbol Device:L
- added R187: 1M, Resistor_SMD:R_0603_1608Metric, symbol Device:R
- added R301, R302, R303, R304: 10k, Resistor_SMD:R_0603_1608Metric, symbol Device:R
- added U39: ISOW7741, Package_SO:SOIC-20W_7.5x12.8mm_P1.27mm, symbol Isolator:ISOW7741
- added U40: 74LVC1G04, Package_TO_SOT_SMD:SOT-23-5, symbol 74xGxx:74LVC1G04
- added U41: ITX2405SA, Converter_DCDC:Converter_DCDC_XP_POWER-ITXxxxxSA_THT, symbol Converter_DCDC:ITX2405SA
- added U42: AD5755-1, Package_CSP:LFCSP-64-1EP_9x9mm_P0.5mm_EP5.21x5.21mm, symbol cems_core:AD5755-1
- R166: value 5k11 0.1% -> 10k; MPN 5k11 0.1% -> 10k
- R167: value 10M -> 5k11 0.1%; MPN 10M -> 5k11 0.1%
- R173: value 100R -> 10M; MPN 100R -> 10M
- R176: value 10k -> 100R; MPN 10k -> 100R
- R178: value 250R 0.1% -> 10k; footprint Resistor_SMD:R_1206_3216Metric -> Resistor_SMD:R_0603_1608Metric; MPN Vishay PTN1206 0.4 W, 10 ppm/K thin film -> 10k
- R180: value 100k -> 250R 0.1%; footprint Resistor_SMD:R_0603_1608Metric -> Resistor_SMD:R_1206_3216Metric; MPN 100k -> Vishay PTN1206 0.4 W, 10 ppm/K thin film
- R181: value 240R 1% -> 100k; MPN 240R 1% -> 100k
- R182: value 2k26 1% -> 240R 1%; MPN 2k26 1% -> 240R 1%
- R183: value 3k -> 2k26 1%; MPN 3k -> 2k26 1%
- R184: value 100k 0.1% -> 3k; MPN 100k 0.1% -> 3k
- R186: value 1M -> 100k 0.1%; MPN 1M -> 100k 0.1%
Connections:
- net +10V_FLOW: now also R185.1; no longer R184.1
- net +13V_AI: now also R182.1; no longer R181.1
- net +24V: now also C307.1, U41.2 (+Vin)
- net +24V_AI: now also C328.1, U42.19 (AVDD)
- net +3V3: now also R165.1, R177.1, C301.1, C304.1, R301.1, U39.1 (V_{IO}), U40.5 (VCC); no longer R176.1
- net +3V3_T: now also R166.1; no longer R165.1
- net +5V: now also C302.1, C303.1, U39.9 (V_{DD})
- net +5V_AI: now also R178.1; no longer R177.1
- net AI5_IN: now also R179.1; no longer R178.1
- net AI6_IN: now also R180.1; no longer R179.1
- net AI_ADJ: now also R182.2, R183.1; no longer R181.2, R182.1
- net AI_ENFLT: now also R177.2; no longer R176.2
- net AI_ERR: now also R178.2; no longer R177.2
- net FLOW_ILIM: now also R184.1; no longer R183.1
- net FLOW_SIG: now also R187.1; no longer R186.1
- net GND: now also C301.2, C302.2, C303.2, C304.2, C307.2, U39.10 (GND1), U39.6 (GNDIO), U40.3 (GND), U41.1 (-Vin)
- net GND_AI: now also R181.2, R184.2, C305.2, C306.2, C308.2, C309.2, C310.2, C311.2, C312.2, C313.2, C314.2, C315.2, C316.2, C317.2, C318.2, C319.2, C320.2, C321.2, C322.2, C323.2, C324.2, C325.2, C326.2, C327.2, C328.2, C329.2, D55.2 (A), D56.2 (A), D57.2 (A), D58.2 (A), J26.2 (Pin_2), J26.4 (Pin_4), J26.6 (Pin_6), J26.8 (Pin_8), R187.2, U39.11 (GND2), U39.15 (GISOIN), U41.7 (-Vout), U42.12 (DGND), U42.13 (~{LDAC}), U42.14 (CLEAR), U42.17 (POC), U42.27 (AVSS), U42.3 (REFGND), U42.35 (AGND), U42.37 (GNDSWB), U42.38 (GNDSWA), U42.4 (REFGND), U42.40 (AVSS), U42.42 (GNDSWD), U42.43 (GNDSWC), U42.5 (AD0), U42.53 (AVSS), U42.6 (AD1), U42.65 (EP); no longer R178.2, R182.2, R185.2
- net GND_T: now also R167.2; no longer R166.2
- net LVL_SIG: now also R181.1; no longer R180.1
- net SPI4_MISO: now also U39.5 (OUTD)
- net SPI4_MOSI: now also U39.3 (INB)
- net SPI4_SCK: now also U39.2 (INA)
- net T1_N: now also R168.1; no longer R167.1
- net T2_N: now also R169.1; no longer R168.1
- net T3_N: now also R170.1; no longer R169.1
- net T4_N: now also R171.1; no longer R170.1
- net T5_N: now also R172.1; no longer R171.1
- net T6_N: now also R173.1; no longer R172.1
- net T_AINCOM: now also R173.2; no longer R167.2
- net T_ENFLT: now also R165.2
- net T_REFP: now also R167.1, R176.2; no longer R166.1, R173.2
- net T_RST: now also R166.2; no longer R165.2
- net T_RTN1: now also R174.1; no longer R173.1
- net T_RTN2: now also R175.1; no longer R174.1
- net T_RTN3: now also R176.1; no longer R175.1
- net V10_MON: now also R185.2, R186.1; no longer R184.2, R185.1
- new net +5V_AO: C308.1, C309.1, C327.1, L4.1, L5.1, L6.1, L7.1, U41.6 (+Vout), U42.45 (AVCC)
- new net +5V_AOD: C305.1, C306.1, C326.1, R302.1, R303.1, R304.1, U39.12 (V_{ISOOUT}), U39.13 (VSEL), U39.14 (EN_IO2), U39.20 (V_{ISOIN}), U42.11 (DVDD)
- new net AO_ALERT: R303.2, U42.15 (~{ALERT})
- new net AO_COMP1: C312.1, U42.23 (COMPDCDC_A)
- new net AO_COMP2: C316.1, U42.32 (COMPDCDC_B)
- new net AO_COMP3: C320.1, U42.48 (COMPDCDC_C)
- new net AO_COMP4: C324.1, U42.57 (COMPDCDC_D)
- new net AO_CS: U39.17 (OUTC), U42.7 (~{SYNC})
- new net AO_DIN: U39.18 (OUTB), U42.9 (SDIN)
- new net AO_DOUT: U39.16 (IND), U42.10 (SDO)
- new net AO_EN1: U39.7 (EN_IO1), U40.4
- new net AO_ENFLT: R301.2, U39.8 (EN/FLT)
- new net AO_FAULT: R304.2, U42.16 (~{FAULT})
- new net AO_IOUT1: C313.1, D55.1 (K), J26.1 (Pin_1), U42.26 (IOUT_A)
- new net AO_IOUT2: C317.1, D56.1 (K), J26.3 (Pin_3), U42.33 (IOUT_B)
- new net AO_IOUT3: C321.1, D57.1 (K), J26.5 (Pin_5), U42.47 (IOUT_C)
- new net AO_IOUT4: C325.1, D58.1 (K), J26.7 (Pin_7), U42.54 (IOUT_D)
- new net AO_REF: C329.1, U42.61 (REFIN), U42.62 (REFOUT)
- new net AO_RST: R302.2, U42.18 (~{RESET})
- new net AO_SCLK: U39.19 (OUTA), U42.8 (SCLK)
- new net AO_SW1: D51.2 (A), L4.2, U42.39 (SWA)
- new net AO_SW2: D52.2 (A), L5.2, U42.36 (SWB)
- new net AO_SW3: D53.2 (A), L6.2, U42.44 (SWC)
- new net AO_SW4: D54.2 (A), L7.2, U42.41 (SWD)
- new net AO_VB1: C310.1, C311.1, D51.1 (K), U42.24 (VBOOST_A)
- new net AO_VB2: C314.1, C315.1, D52.1 (K), U42.34 (VBOOST_B)
- new net AO_VB3: C318.1, C319.1, D53.1 (K), U42.46 (VBOOST_C)
- new net AO_VB4: C322.1, C323.1, D54.1 (K), U42.56 (VBOOST_D)
- new net CS_AO: U39.4 (INC), U40.2
- no-connect marks 19 -> 40
Other:
- note added: "C316: NOT FITTED. D56: NOT FITTED. C317: NOT FITTED. L6: NOT FITTED. D53: NOT FITTED. C318: NOT FITTED. C319: NOT FITTED. C320: NOT FITTED. D57: NOT FITTED. C321: NOT FITTED. L7: NOT FITTED. D54: NOT FITTED. C322: NOT FITTED. C323: NOT FITTED. C324: NOT FITTED. D58: NOT FITTED. C325: NOT FITTED. U42: NOT FITTED. 4 x 4-20 mA, short and open-loop detect. Pin numbers from Table 5 (31 Oct). VOUT/+VSE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"
- note added: "Notes U28: VSEL to GND2 = 3.3 V out (140 mA) R165: EN/FLT high (VIO level) enables the DC/DC; reads low on a fault U30: pinout checked (SBAS660, 31 Oct). Internal 4.096 MHz clock (CLK to DGND), START low (conversions by command), DOUT/DRDY on one pin C145: REFOUT to REFCOM R167: RTD reference resistor, 10 ppm/K C147: CHECK AINCOM and the TC bias against the io-node schematic C148: differential fi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"
- note added: "R185: 10 V monitor for ratiometric correction D49: clamps +5V_LVL D50: clamps +10V_FLOW (12.2 V min breakdown) J25: level (DFRobot SEN0205): 5 V, SIG, 0 V; mass flow (AWM5104VN): +10 V, OUT, 0 V U40: NOT FITTED. C301: NOT FITTED. U39: NOT FITTED. VSEL to VISOOUT = 5 V out (DVDD) R301: NOT FITTED. EN/FLT high (VIO level) enables the DC/DC; reads low on a fault C302: NOT FITTED. C303: NOT FITTED. C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"
- note removed: "J21: T5 +/-, T6 +/-, RTD return U31: VSEL to VISOOUT = 5 V out (110 mA) R176: EN/FLT high (VIO level) enables the DC/DC; reads low on a fault U33: loop power 6 x 22 mA + level + mass-flow supply, about 4 W U34: internal oscillator and 2.5 V reference. VIN0/1: 4-20 mA ch 5/6 on shunts; VIN2 level; VIN3 mass flow; VIN4 10 V monitor; VIN5 5 V monitor. Pinout checked (31 Oct); CHECK the exposed pad s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"
- note removed: "J24: per channel: 24 V loop, IN, 0 V (2-wire or 4-wire transmitters) U35: level sensor 5 V, internal current limit R180: defined level when unplugged U36: 13 V pre-regulator, about 0.5 W: copper on the VO pins R182: 1.25 x (1 + 2260/240) = 13.0 V U38: SET driven by the REF5010 (no RSET). CHECK PGFB tie when PG is unused R183: about 50 mA current limit R184: 10 V monitor for ratiometric correction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"
- note removed: "Notes U28: VSEL to GND2 = 3.3 V out (140 mA) R164: EN/FLT high (VIO level) enables the DC/DC; reads low on a fault U30: pinout checked (SBAS660, 31 Oct). Internal 4.096 MHz clock (CLK to DGND), START low (conversions by command), DOUT/DRDY on one pin C145: REFOUT to REFCOM R166: RTD reference resistor, 10 ppm/K C147: CHECK AINCOM and the TC bias against the io-node schematic C148: differential fi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"
- moved on the sheet: C154, C155, C156, C157, C158, C159, C160, C161, C162, C163, C164, C165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
