File: hardware/core_pcb/io_ana.kicad_sch (KiCad schematic)
At the start: 141 parts, among them J19 TEMP1, J20 TEMP2, J21 TEMP3, J22 AI 1-2, J23 AI 3-4, J24 AI 5-6, J25 SENSORS, J26 AO 1-4, U28 ISOW7741, U29 74LVC1G04, U30 ADS124S08, U31 ISOW7741, U32 74LVC1G04, U33 ITX2424SA, U34 AD4112, U35 L78L05, U36 LM317L, U37 REF5010, U38 LT3045, U39 ISOW7741, U40 74LVC1G04, U41 ITX2405SA, U42 AD5755-1

Commit message: CORE PCB: SPI expansion header J26 for plug-on modules; analog outputs move off the core
Gary: analog out as an add-on module. J26 10-way latched IDC: +24 V and +3.3 V behind PTCs,
SPI4 through 100R, MISO buffered by a 74LVC1G125 enabled by CS_EXP (PD3), EXP_INT on PD7.
The AD5755-1 block drafted in 04adb9f is removed from the core and will become the module.
Layout block plan fits again. CORE_PCB.md section 16.

Co-Authored-By: Claude Opus 5.5 <noreply@anthropic.com>
Claude-Session: https://claude.ai/code/session_014onnq3eRiDkqdAB6fKiRDW
Parts:
- removed C136, C301, C303, C304, C306, C309, C326, C329: 100n, Capacitor_SMD:C_0603_1608Metric, symbol Device:C
- removed C137, C302, C305, C327: 10u, Capacitor_SMD:C_0805_2012Metric, symbol Device:C
- removed C307: 10u 50V, Capacitor_SMD:C_1210_3225Metric, symbol Device:C
- removed C308: 22u, Capacitor_SMD:C_1210_3225Metric, symbol Device:C
- removed C310, C314, C318, C322: 4u7 50V, Capacitor_SMD:C_1210_3225Metric, symbol Device:C
- removed C311, C315, C319, C323, C328: 100n 50V, Capacitor_SMD:C_0603_1608Metric, symbol Device:C
- removed C312, C316, C320, C324: 10n, Capacitor_SMD:C_0603_1608Metric, symbol Device:C
- removed C313, C317, C321, C325: 4n7 50V, Capacitor_SMD:C_0603_1608Metric, symbol Device:C
- removed D51, D52, D53, D54: PMEG4010, Diode_SMD:D_SOD-323F, symbol Device:D_Schottky
- removed D55, D56, D57, D58: SMAJ33A, Diode_SMD:D_SMA, symbol Device:D_Zener
- removed J26: AO 1-4, Connector_Phoenix_MC:PhoenixContact_MCV_1,5_8-G-3.5_1x08_P3.50mm_Vertical, symbol Connector_Generic:Conn_01x08
- removed L4, L5, L6, L7: 10uH, Inductor_SMD:L_Coilcraft_XAL4040-XXX, symbol Device:L
- removed R165, R166, R301, R302, R303, R304: 10k, Resistor_SMD:R_0603_1608Metric, symbol Device:R
- removed R167: 5k11 0.1%, Resistor_SMD:R_0603_1608Metric, symbol Device:R
- removed R168, R169: 10M, Resistor_SMD:R_0603_1608Metric, symbol Device:R
- removed U39: ISOW7741, Package_SO:SOIC-20W_7.5x12.8mm_P1.27mm, symbol Isolator:ISOW7741
- removed U40: 74LVC1G04, Package_TO_SOT_SMD:SOT-23-5, symbol 74xGxx:74LVC1G04
- removed U41: ITX2405SA, Converter_DCDC:Converter_DCDC_XP_POWER-ITXxxxxSA_THT, symbol Converter_DCDC:ITX2405SA
- removed U42: AD5755-1, Package_CSP:LFCSP-64-1EP_9x9mm_P0.5mm_EP5.21x5.21mm, symbol cems_core:AD5755-1
- added C176: 4u7 25V, Capacitor_SMD:C_0805_2012Metric, symbol Device:C
- added C177: 10u 25V, Capacitor_SMD:C_0805_2012Metric, symbol Device:C
- added R188: 2k26 1%, Resistor_SMD:R_0603_1608Metric, symbol Device:R
- added R189: 3k, Resistor_SMD:R_0603_1608Metric, symbol Device:R
- added R190, R191: 100k 0.1%, Resistor_SMD:R_0603_1608Metric, symbol Device:R
- added R192: 1M, Resistor_SMD:R_0603_1608Metric, symbol Device:R
- C139, C142, C157: value 100n -> 10u; footprint Capacitor_SMD:C_0603_1608Metric -> Capacitor_SMD:C_0805_2012Metric; MPN 100n -> 10u
- C140, C158: value 10u -> 100n; footprint Capacitor_SMD:C_0805_2012Metric -> Capacitor_SMD:C_0603_1608Metric; MPN 10u -> 100n
- C143, C170: value 1u -> 100n; MPN 1u -> 100n
- C147: value 100n -> 1u; MPN 100n -> 1u
- C148, C149: value 10n C0G -> 100n; MPN 10n C0G -> 100n
- C154: value 100n -> 10n C0G; MPN 100n -> 10n C0G
- C155: value 10u -> 10n C0G; footprint Capacitor_SMD:C_0805_2012Metric -> Capacitor_SMD:C_0603_1608Metric; MPN 10u -> 10n C0G
- C160: value 10u 50V -> 10u; footprint Capacitor_SMD:C_1210_3225Metric -> Capacitor_SMD:C_0805_2012Metric; MPN 10u 50V -> 10u
- C161: value 10u 50V -> 100n; footprint Capacitor_SMD:C_1210_3225Metric -> Capacitor_SMD:C_0603_1608Metric; MPN 10u 50V -> 100n
- C162: value 100n -> 10u 50V; footprint Capacitor_SMD:C_0603_1608Metric -> Capacitor_SMD:C_1210_3225Metric; MPN 100n -> 10u 50V
- C163: value 1u -> 10u 50V; footprint Capacitor_SMD:C_0603_1608Metric -> Capacitor_SMD:C_1210_3225Metric; MPN 1u -> 10u 50V
- C169: value 330n 50V -> 1u; MPN 330n 50V -> 1u
- C171: value 1u 25V -> 330n 50V; footprint Capacitor_SMD:C_0805_2012Metric -> Capacitor_SMD:C_0603_1608Metric; MPN 1u 25V -> 330n 50V
- C174: value 4u7 25V -> 1u; footprint Capacitor_SMD:C_0805_2012Metric -> Capacitor_SMD:C_0603_1608Metric; MPN 4u7 25V -> 1u
- C175: value 10u 25V -> 1u 25V; MPN 10u 25V -> 1u 25V
- R170, R171: value 10M -> 10k; MPN 10M -> 10k
- R172: value 10M -> 5k11 0.1%; MPN 10M -> 5k11 0.1%
- R174, R175, R176: value 100R -> 10M; MPN 100R -> 10M
- R177, R178: value 10k -> 10M; MPN 10k -> 10M
- R179, R180: value 250R 0.1% -> 100R; footprint Resistor_SMD:R_1206_3216Metric -> Resistor_SMD:R_0603_1608Metric; MPN Vishay PTN1206 0.4 W, 10 ppm/K thin film -> 100R
- R181: value 100k -> 100R; MPN 100k -> 100R
- R182: value 240R 1% -> 10k; MPN 240R 1% -> 10k
- R183: value 2k26 1% -> 10k; MPN 2k26 1% -> 10k
- R184: value 3k -> 250R 0.1%; footprint Resistor_SMD:R_0603_1608Metric -> Resistor_SMD:R_1206_3216Metric; MPN 3k -> Vishay PTN1206 0.4 W, 10 ppm/K thin film
- R185: value 100k 0.1% -> 250R 0.1%; footprint Resistor_SMD:R_0603_1608Metric -> Resistor_SMD:R_1206_3216Metric; MPN 100k 0.1% -> Vishay PTN1206 0.4 W, 10 ppm/K thin film
- R186: value 100k 0.1% -> 100k; MPN 100k 0.1% -> 100k
- R187: value 1M -> 240R 1%; MPN 1M -> 240R 1%
Connections:
- net +10V_FLOW: now also C177.1, R190.1; no longer C175.1, R185.1
- net +13V_AI: now also C173.1, R187.1, C176.1; no longer C171.1, C174.1, R182.1
- net +24V: now also C162.1; no longer C160.1
- net +24V_AI: now also C163.1, C171.1; no longer C161.1, C169.1
- net +3V3: now also C138.1, C141.1, C156.1, C159.1, R170.1, R182.1; no longer C139.1, C154.1, C157.1, R177.1
- net +3V3_T: now also C143.1, C144.1, R171.1; no longer C140.1, C141.1
- net +3V3_TA: now also C145.1, C146.1; no longer C143.1, C144.1
- net +5V: now also C139.1, C140.1, C157.1, C158.1; no longer C138.1, C155.1, C156.1
- net +5V_AI: now also C160.1, C161.1, C164.1, R183.1; no longer C158.1, C159.1, C162.1, R178.1
- net +5V_AIA: now also C165.1, C166.1; no longer C163.1, C164.1
- net +5V_LVL: now also C172.1; no longer C170.1
- net AI5_IN: now also R184.1; no longer R179.1
- net AI6_IN: now also R185.1; no longer R180.1
- net AI_ADJ: now also R187.2, R188.1; no longer R182.2, R183.1
- net AI_ENFLT: now also R182.2; no longer R177.2
- net AI_ERR: now also R183.2; no longer R178.2
- net AI_REF: now also C170.1; no longer C168.1
- net AI_REGCAPA: now also C167.1, C168.1; no longer C165.1, C166.1
- net AI_REGCAPD: now also C169.1; no longer C167.1
- net FLOW_ILIM: now also R189.1; no longer R184.1
- net FLOW_SIG: now also R192.1; no longer R187.1
- net GND: now also C140.2, C141.2, C158.2, C159.2, C162.2; no longer C154.2, C155.2, C160.2
- net GND_AI: now also C160.2, R185.2, C176.2, C177.2, R188.2, R189.2, R191.2, R192.2; no longer C158.2, C159.2, C162.2, R179.2, R180.2, R181.2, R183.2, R187.2
- net GND_T: now also C148.2, C149.2, R172.2; no longer C140.2, C141.2
- net LVL_SIG: now also R186.1; no longer R181.1
- net REF10: now also C175.1; no longer C173.1
- net REF10_NR: now also C174.1; no longer C172.1
- net T1_N: now also C150.2, R173.1; no longer C148.2
- net T1_P: now also C150.1; no longer C148.1
- net T2_N: now also C151.2, R174.1; no longer C149.2
- net T2_P: now also C151.1; no longer C149.1
- net T3_N: now also C152.2, R175.1; no longer C150.2, R170.1
- net T3_P: now also C152.1; no longer C150.1
- net T4_N: now also C153.2, R176.1; no longer C151.2, R171.1
- net T4_P: now also C153.1; no longer C151.1
- net T5_N: now also C154.2, R177.1; no longer C152.2, R172.1
- net T5_P: now also C154.1; no longer C152.1
- net T6_N: now also C155.2, R178.1; no longer C153.2, R173.1
- net T6_P: now also C155.1; no longer C153.1
- net T_AINCOM: now also C149.1, R174.2, R175.2, R176.2, R177.2, R178.2; no longer C147.1, R170.2, R171.2, R172.2
- net T_ENFLT: now also R170.2
- net T_REFOUT: now also C147.1; no longer C145.1
- net T_REFP: now also C148.1, R172.1, R179.2, R180.2, R181.2; no longer C146.1, R174.2, R175.2, R176.2
- net T_RST: now also R171.2
- net T_RTN1: now also R179.1; no longer R174.1
- net T_RTN2: now also R180.1; no longer R175.1
- net T_RTN3: now also R181.1; no longer R176.1
- net V10_MON: now also R190.2, R191.1; no longer R185.2, R186.1
- no-connect marks 40 -> 19
Other:
- note added: "J21: T5 +/-, T6 +/-, RTD return U31: VSEL to VISOOUT = 5 V out (110 mA) R182: EN/FLT high (VIO level) enables the DC/DC; reads low on a fault U33: loop power 6 x 22 mA + level + mass-flow supply, about 4 W U34: internal oscillator and 2.5 V reference. VIN0/1: 4-20 mA ch 5/6 on shunts; VIN2 level; VIN3 mass flow; VIN4 10 V monitor; VIN5 5 V monitor. Pinout checked (31 Oct); CHECK the exposed pad s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"
- note added: "J24: per channel: 24 V loop, IN, 0 V (2-wire or 4-wire transmitters) U35: level sensor 5 V, internal current limit R186: defined level when unplugged U36: 13 V pre-regulator, about 0.5 W: copper on the VO pins R188: 1.25 x (1 + 2260/240) = 13.0 V U38: SET driven by the REF5010 (no RSET). CHECK PGFB tie when PG is unused R189: about 50 mA current limit R190: 10 V monitor for ratiometric correction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"
- note added: "Notes U28: VSEL to GND2 = 3.3 V out (140 mA) R170: EN/FLT high (VIO level) enables the DC/DC; reads low on a fault U30: pinout checked (SBAS660, 31 Oct). Internal 4.096 MHz clock (CLK to DGND), START low (conversions by command), DOUT/DRDY on one pin C147: REFOUT to REFCOM R172: RTD reference resistor, 10 ppm/K C149: CHECK AINCOM and the TC bias against the io-node schematic C150: differential fi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"
- note removed: "C316: NOT FITTED. D56: NOT FITTED. C317: NOT FITTED. L6: NOT FITTED. D53: NOT FITTED. C318: NOT FITTED. C319: NOT FITTED. C320: NOT FITTED. D57: NOT FITTED. C321: NOT FITTED. L7: NOT FITTED. D54: NOT FITTED. C322: NOT FITTED. C323: NOT FITTED. C324: NOT FITTED. D58: NOT FITTED. C325: NOT FITTED. U42: NOT FITTED. 4 x 4-20 mA, short and open-loop detect. Pin numbers from Table 5 (31 Oct). VOUT/+VSE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"
- note removed: "Notes U28: VSEL to GND2 = 3.3 V out (140 mA) R165: EN/FLT high (VIO level) enables the DC/DC; reads low on a fault U30: pinout checked (SBAS660, 31 Oct). Internal 4.096 MHz clock (CLK to DGND), START low (conversions by command), DOUT/DRDY on one pin C145: REFOUT to REFCOM R167: RTD reference resistor, 10 ppm/K C147: CHECK AINCOM and the TC bias against the io-node schematic C148: differential fi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"
- note removed: "R185: 10 V monitor for ratiometric correction D49: clamps +5V_LVL D50: clamps +10V_FLOW (12.2 V min breakdown) J25: level (DFRobot SEN0205): 5 V, SIG, 0 V; mass flow (AWM5104VN): +10 V, OUT, 0 V U40: NOT FITTED. C301: NOT FITTED. U39: NOT FITTED. VSEL to VISOOUT = 5 V out (DVDD) R301: NOT FITTED. EN/FLT high (VIO level) enables the DC/DC; reads low on a fault C302: NOT FITTED. C303: NOT FITTED. C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"
- moved on the sheet: C138, C139, C140, C141, C142, C143, C144, C145, C146, C147, C148, C149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
