File: hardware/core_pcb/io_dig.kicad_sch (KiCad schematic)
At the start: 94 parts, among them J10 BANK A IDC26, J11 BANK B, J12 INPUTS IDC26, U11 MAX6369, U12 74LVC1G08, U13 74LVC1G04, U14 ISO2H823V2.5, U15 ISO808A-1, U16 ISO1I813T

Commit message: CORE PCB: layout start in BC 215,6 outline; breakout header and carrier chosen
gen_pcb.py writes cems_core.kicad_pcb from design.py: 4 layers, assumed BC 215,6
outline (211.5 x 85.1 mm; BC 161,6 is too small for the I/O section), all 423
footprints with nets, connectors on the housing faces, a block plan per sheet, net
classes and 2.5 mm isolation rules between the four ground domains. Placeholder
PG-VQFN-70 footprint for the ISO2H823V2.5 (to redraw). Breakout: Wurth 61202622821
latched header, board 50 x 80 mm for a standard DIN PCB holder.

Co-Authored-By: Claude Opus 5.5 <noreply@anthropic.com>
Claude-Session: https://claude.ai/code/session_014onnq3eRiDkqdAB6fKiRDW
Parts:
- J10: MPN 26-way shrouded latched box header, same as the breakout (h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 -> Wurth 61202622821 (WR-BHD, long latches, 3 A), same as the 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
- J12: MPN 26-way shrouded latched box header, same as J10 -> Wurth 61202622821, same as J10
Changed lines of the file:
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@@
       (effects (font (size 1.27 1.27)) hide)
     )
-    (property "MPN" "26-way shrouded latched box header, same as the breakout (hardware/io_breakout)" (id 4) (at 528.32 35.56 0)
+    (property "MPN" "Wurth 61202622821 (WR-BHD, long latches, 3 A), same as the breakout" (id 4) (at 528.32 35.56 0)
       (effects (font (size 1.27 1.27)) hide)
     )
@@
       (effects (font (size 1.27 1.27)) hide)
     )
-    (property "MPN" "26-way shrouded latched box header, same as J10" (id 4) (at 35.56 309.88 0)
-      (effects (font (size 1.27 1.27)) hide)
-    )
+    (property "MPN" "Wurth 61202622821, same as J10" (id 4) (at 35.56 309.88 0)
+      (effects (font (size 1.27 1.27)) hide)
+    )

Commit message: CORE PCB: I/O chip pinouts checked against datasheets; gate latch, ODIS polarity
Pin tables of AD4112, ADS124S08, ISO2H823V2.5, ISO1I813T, ISO808A-1, ISO7741 and
ISOW7741 compared with the datasheets: all match. Fixes from the check: ISO2H823 /ODIS
is active low (takes GATE directly); OLADJ fitted 12.1k; CLKADJ 10k 0.1 %; ROSC 22.1k;
ISOW7741 EN/FLT pulled to 3.3 V; MAX6369 WDO only pulses, so a 74LVC1G175 latches a
trip until GATE_EN is re-armed. hardware/datasheets/IO_CHIPS_DATASHEET_CHECK.md holds the
extracts and the AD4112 register facts for the driver.

Co-Authored-By: Claude Opus 5.5 <noreply@anthropic.com>
Claude-Session: https://claude.ai/code/session_014onnq3eRiDkqdAB6fKiRDW
Parts:
- R104: value 10k -> 10k 0.1%; MPN 10k -> 10k 0.1%
- R106: value DNF -> 12k1 1%; MPN DNF -> 12k1 1%; now fitted
- R118: value 22k 1% -> 22k1 1%; MPN 22k 1% -> 22k1 1%
- U13: value 74LVC1G04 -> 74LVC1G175; footprint Package_TO_SOT_SMD:SOT-23-5 -> Package_TO_SOT_SMD:SOT-23-6; symbol 74xGxx:74LVC1G04 -> 74xGxx:74LVC1G175; MPN SN74LVC1G04DBVR -> SN74LVC1G175DBVR
Connections:
- net +3V3: now also U13.3 (D)
- net GATE: now also U14.40 (ODIS); no longer U13.2
- net GATE_EN: now also U13.1 (C)
- net GND: now also U13.2 (GND); no longer U13.3 (GND)
- net WDO_N: now also U13.6 (~{CLR}); no longer U12.2
- net GATE_N renamed GATE_ARM
- net GATE_ARM: now also U12.2; no longer U14.40 (ODIS)
Other:
- note added: "D46: NOT FITTED. D47: NOT FITTED. D48: NOT FITTED. U16: serial mode; internal DC/DC off (DC_ENA low), field side from VBB. Values from Infineon's ISO1I813T evaluation board. Pinout checked against the datasheet (31 Oct): serial mode 3 (24-bit, CRC) R118: 22.1k: about 500 kHz scan (datasheet typical) R119: type 1 (eval board RTS = 33 ohm; datasheet: type 2 = 33k, type 3 = 330k). CHECK type 1 value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"
- note added: "J10: same pinout as the breakout J1, straight-through ribbon F10: ribbon +24 V (breakout LEDs) U15: pinout checked against DS14170 (31 Oct). Tab = VCC (+24V_FB): copper pour on the field side only C200: bank B bulk J11: 8 A return over 2 contacts: CHECK the plug rating (8 A per contact) D31: flyback at the terminal, as on the breakout D41: NOT FITTED. fast-release option (remove the 0R) D42: NOT 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"
- note added: "Notes U11: SET2..0 = 010: 30 ms startup delay and timeout (minimum), so outputs drop within 50 ms. WDO pulses; U13 latches it R102: gate shut while the MCU is in reset U13: D flip-flop: rising GATE_EN sets GATE_ARM, a watchdog trip clears it until the next rising edge U12: GATE = GATE_EN and armed (no watchdog trip since) R103: firmware reads the gate back (PD8) U14: pinout checked against datash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"
- note removed: "D47: NOT FITTED. D48: NOT FITTED. U16: serial mode; internal DC/DC off (DC_ENA low), field side from VBB. Values from Infineon's ISO1I813T evaluation board. CHECK pinout and SEL/MS levels R118: 500 kHz R119: type 1/3 (eval board RTS). CHECK R120: wire-break threshold (eval board). CHECK R122: RIN, eval board R123: RLED (no LED here; the breakout has them) J12: same pinout as the breakout J1 F11: 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"
- note removed: "F10: ribbon +24 V (breakout LEDs) U15: tab = VCC (+24V_FB): copper pour on the field side only. CHECK pinout C200: bank B bulk J11: 8 A return over 2 contacts: CHECK the plug rating (8 A per contact) D31: flyback at the terminal, as on the breakout D41: NOT FITTED. fast-release option (remove the 0R) D42: NOT FITTED. D43: NOT FITTED. D44: NOT FITTED. D45: NOT FITTED. D46: NOT FITTED."
- note removed: "Notes U11: SET2..0 = 010: 30 ms watchdog (outputs off within 50 ms). CHECK the SET table and startup delay R102: gate shut while the MCU is in reset U12: GATE = GATE_EN and watchdog OK R103: firmware reads the gate back (PD8) U13: ODIS of the ISO2H823V2.5. CHECK ODIS polarity: if it is active low, link GATE instead U14: serial mode: SEL high, MS0/MS1 high, ALE/RST low. No LED matrix: X pins tied,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"
- moved on the sheet: C102, C103, C104, C105, C106, C107, C108, C109, C110, C111, C112, C113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

Commit message: One 40-way ribbon for all digital I/O (Gary, 31 Oct)
Main board: J10 becomes a 40-way latched IDC header carrying bank A outputs 1-8 (pins
1-16, each beside its 0 V) and inputs 1-8 (pins 17-32), with 4 x +24 V and 4 x 0 V; J12
and F11 removed, so no ribbon can go into the wrong slot. Breakout rev 0.2: one board,
50 x 80 mm, two-tier 3.81 mm pluggable headers (valves OUT over 0V, inputs IN over +24V,
plus a 0V strip for 3-wire sensors), LEDs on every channel, flyback options on the valves.
Two-tier footprint is a placeholder until the maker's drawing is checked.

Co-Authored-By: Claude Opus 5.5 <noreply@anthropic.com>
Claude-Session: https://claude.ai/code/session_014onnq3eRiDkqdAB6fKiRDW
Parts:
- removed F11: 0.75A, Fuse:Fuse_1812_4532Metric, symbol Device:Polyfuse
- removed J12: INPUTS IDC26, Connector_IDC:IDC-Header_2x13_P2.54mm_Latch_Vertical, symbol Connector_Generic:Conn_02x13_Odd_Even
- J10: value BANK A IDC26 -> DIGITAL I/O IDC40; footprint Connector_IDC:IDC-Header_2x13_P2.54mm_Latch_Vertical -> Connector_IDC:IDC-Header_2x20_P2.54mm_Latch_Vertical; symbol Connector_Generic:Conn_02x13_Odd_Even -> Connector_Generic:Conn_02x20_Odd_Even; MPN Wurth 61202622821 (WR-BHD, long latches, 3 A), same as the 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 -> Wurth 61204022821 (WR-BHD 40-way, long latches, 3 A). CHECK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
Connections:
- net DI1: now also J10.17 (Pin_17)
- net DI2: now also J10.19 (Pin_19)
- net DI3: now also J10.21 (Pin_21)
- net DI4: now also J10.23 (Pin_23)
- net DI5: now also J10.25 (Pin_25)
- net DI6: now also J10.27 (Pin_27)
- net DI7: now also J10.29 (Pin_29)
- net DI8: now also J10.31 (Pin_31)
- net FIELD_0V: now also J10.28 (Pin_28), J10.30 (Pin_30), J10.32 (Pin_32), J10.34 (Pin_34), J10.36 (Pin_36), J10.38 (Pin_38), J10.40 (Pin_40)
- removed net +24V_RA: F10.2, J10.17 (Pin_17), J10.19 (Pin_19), J10.21 (Pin_21), J10.23 (Pin_23), J10.25 (Pin_25)
- new net +24V_RIB: F10.2, J10.33 (Pin_33), J10.35 (Pin_35), J10.37 (Pin_37), J10.39 (Pin_39)
Other:
- note added: "D48: NOT FITTED. U16: serial mode; internal DC/DC off (DC_ENA low), field side from VBB. Values from Infineon's ISO1I813T evaluation board. Pinout checked against the datasheet (31 Oct): serial mode 3 (24-bit, CRC) R118: 22.1k: about 500 kHz scan (datasheet typical) R119: type 1 (eval board RTS = 33 ohm; datasheet: type 2 = 33k, type 3 = 330k). CHECK type 1 value R120: wire-break current, 25-55k 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"
- note added: "U15: pinout checked against DS14170 (31 Oct). Tab = VCC (+24V_FB): copper pour on the field side only C200: bank B bulk J11: 8 A return over 2 contacts: CHECK the plug rating (8 A per contact) D31: flyback at the terminal, as on the breakout D41: NOT FITTED. fast-release option (remove the 0R) D42: NOT FITTED. D43: NOT FITTED. D44: NOT FITTED. D45: NOT FITTED. D46: NOT FITTED. D47: NOT FITTED."
- note removed: "D46: NOT FITTED. D47: NOT FITTED. D48: NOT FITTED. U16: serial mode; internal DC/DC off (DC_ENA low), field side from VBB. Values from Infineon's ISO1I813T evaluation board. Pinout checked against the datasheet (31 Oct): serial mode 3 (24-bit, CRC) R118: 22.1k: about 500 kHz scan (datasheet typical) R119: type 1 (eval board RTS = 33 ohm; datasheet: type 2 = 33k, type 3 = 330k). CHECK type 1 value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"
- note removed: "J10: same pinout as the breakout J1, straight-through ribbon F10: ribbon +24 V (breakout LEDs) U15: pinout checked against DS14170 (31 Oct). Tab = VCC (+24V_FB): copper pour on the field side only C200: bank B bulk J11: 8 A return over 2 contacts: CHECK the plug rating (8 A per contact) D31: flyback at the terminal, as on the breakout D41: NOT FITTED. fast-release option (remove the 0R) D42: NOT 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"
- moved on the sheet: C118, C119, C120, C121, C122, C123, C124, C200, D31, D32, D33, D34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

Commit message: CORE PCB + breakout: make every user plug fit only its own header
Three pitch families (5.08 power/24 V outputs, 3.81 bank B, 3.5 sensors), one size per
header except the harmless temperature and 4-20 mA groups, and a coding key per header
(script-checked against every plug and shift). J13+J14 merged into one 4-way field plug;
pump power and signals on one 6-way plug (J16 gone); relays 3-way. Survival layer: 1k 1 W
pump outputs, per-channel relay PTCs + CPC1014N, 30 mA loop current limiters, TVS on the
5 V and 10 V sensor supplies. CORE_PCB.md section 15 has the mis-plug tables.

Co-Authored-By: Claude Opus 5.5 <noreply@anthropic.com>
Claude-Session: https://claude.ai/code/session_014onnq3eRiDkqdAB6fKiRDW
Parts:
- J11: MPN Phoenix MCV 1,5/10-G-3,81 (or Degson / Dinkle equivalent) +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 -> Phoenix MCV 1,5/10-G-3,81 + coded, labelled plug
Changed lines of the file:
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@@
       (effects (font (size 1.27 1.27)) hide)
     )
-    (property "MPN" "Phoenix MCV 1,5/10-G-3,81 (or Degson / Dinkle equivalent) + mating plug" (id 4) (at 106.68 154.94 0)
+    (property "MPN" "Phoenix MCV 1,5/10-G-3,81 + coded, labelled plug" (id 4) (at 106.68 154.94 0)
       (effects (font (size 1.27 1.27)) hide)
     )

Commit message: CORE PCB: fit-optional 4 x 4-20 mA analog outputs (AD5755-1, all DNP)
AD5755-1 on the analog island with its own ISOW7741 (CS_AO on PD3) and an ITX2405SA for
the boost converters; keyed 8-way 3.5 mm J26 (keys 2, 6, script-checked). Pin numbers from
the datasheet Table 5. Layout block plan now 2.8 mm over in io_pwr: the board is full
single-sided, see thread for the module option.

Co-Authored-By: Claude Opus 5.5 <noreply@anthropic.com>
Claude-Session: https://claude.ai/code/session_014onnq3eRiDkqdAB6fKiRDW
Parts:
- added R143: 10k, Resistor_SMD:R_0603_1608Metric, symbol Device:R
Connections:
- net +3V3: now also R143.1
- new net CS_AO: R143.2
Changed lines of the file:
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@@
+    )
+  )
+  (global_label "+3V3" (shape passive) (at 71.12 278.13 90) (fields_autoplaced)
+    (effects (font (size 1.27 1.27)) (justify left))
+    (property "Intersheetrefs" "${INTERSHEET_REFS}" (id 0) (at 71.12 278.13 90)
+      (effects (font (size 1.27 1.27)) (justify left) hide)
+    )
+  )
+  (global_label "CS_AO" (shape passive) (at 71.12 285.75 270) (fields_autoplaced)
+    (effects (font (size 1.27 1.27)) (justify right))
+    (property "Intersheetrefs" "${INTERSHEET_REFS}" (id 0) (at 71.12 285.75 270)
+      (effects (font (size 1.27 1.27)) (justify right) hide)
     )
   )
@@
         )
       )
+    )
+  )
+  (symbol (lib_id "Device:R") (at 71.12 281.94 0) (unit 1)
+    (in_bom yes) (on_board yes) (dnp no)
+    (property "Reference" "R143" (id 0) (at 71.12 266.7 0)
+      (effects (font (size 1.27 1.27)))
+    )
+    (property "Value" "10k" (id 1) (at 71.12 299.72 0)
+      (effects (font (size 1.27 1.27)))
+    )
+    (property "Footprint" "Resistor_SMD:R_0603_1608Metric" (id 2) (at 71.12 281.94 0)
+      (effects (font (size 1.27 1.27)) hide)
+    )
+    (property "Datasheet" "~" (id 3) (at 71.12 281.94 0)
+      (effects (font (size 1.27 1.27)) hide)
+    )
+    (property "MPN" "10k" (id 4) (at 71.12 281.94 0)
+      (effects (font (size 1.27 1.27)) hide)
+    )
+    (pin "1")
+    (pin "2")
+    (instances
+      (project "cems_core"
+        (path "/4503b035-ec93-58ad-a08a-2d339f99cb7b/6e0e6d03-f39f-55a0-81fa-cfe9e7b5fa43"
+          (reference "R143") (unit 1)
+        )
+      )

Commit message: CORE PCB: SPI expansion header J26 for plug-on modules; analog outputs move off the core
Gary: analog out as an add-on module. J26 10-way latched IDC: +24 V and +3.3 V behind PTCs,
SPI4 through 100R, MISO buffered by a 74LVC1G125 enabled by CS_EXP (PD3), EXP_INT on PD7.
The AD5755-1 block drafted in 04adb9f is removed from the core and will become the module.
Layout block plan fits again. CORE_PCB.md section 16.

Co-Authored-By: Claude Opus 5.5 <noreply@anthropic.com>
Claude-Session: https://claude.ai/code/session_014onnq3eRiDkqdAB6fKiRDW
Parts:
- added C125: 100n, Capacitor_SMD:C_0603_1608Metric, symbol Device:C
- added C126: 100n, Capacitor_SMD:C_0805_2012Metric, symbol Device:C
- added F23: 0.5A, Fuse:Fuse_1206_3216Metric, symbol Device:Polyfuse
- added F24: 0.1A, Fuse:Fuse_1206_3216Metric, symbol Device:Polyfuse
- added J26: SPI EXPANSION, Connector_IDC:IDC-Header_2x05_P2.54mm_Latch_Vertical, symbol Connector_Generic:Conn_02x05_Odd_Even
- added R144, R145, R146, R147, R148: 10k, Resistor_SMD:R_0603_1608Metric, symbol Device:R
- added U39: 74LVC1G125, Package_TO_SOT_SMD:SOT-23-5, symbol 74xGxx:74LVC1G125
- R138, R139, R140: value 10k -> 100R; MPN 10k -> 100R
- R141: value 10k -> 100k; MPN 10k -> 100k
Connections:
- net CS_AO is gone; now on net CS_A: R143.2
- net +3V3: now also C125.1, F24.1, R144.1, R145.1, R146.1, R147.1, R148.1, U39.5 (VCC); no longer R138.1, R139.1, R140.1, R141.1
- net CS_A: no longer R138.2
- net CS_AI: now also R147.2; no longer R142.2
- net CS_B: now also R144.2; no longer R139.2
- net CS_IN: now also R145.2; no longer R140.2
- net CS_T: now also R146.2; no longer R141.2
- net GND: now also R141.2, C125.2, C126.2, J26.2 (Pin_2), J26.4 (Pin_4), J26.6 (Pin_6), U39.3 (GND)
- net SPI4_MISO: now also U39.4
- net SPI4_MOSI: now also R139.1
- net SPI4_SCK: now also R138.1
- new net +24V: F23.1
- new net +24V_EXP: C126.1, F23.2, J26.1 (Pin_1)
- new net +3V3_EXP: F24.2, J26.3 (Pin_3)
- new net CS_EXP: R140.1, R148.2, U39.1
- new net EXP_CS: J26.9 (Pin_9), R140.2
- new net EXP_INT: J26.10 (Pin_10), R142.2
- new net EXP_MISO: J26.8 (Pin_8), R141.1, U39.2
- new net EXP_MOSI: J26.7 (Pin_7), R139.2
- new net EXP_SCK: J26.5 (Pin_5), R138.2
Other:
- note added: "C200: bank B bulk J11: 8 A return over 2 contacts: CHECK the plug rating (8 A per contact) D31: flyback at the terminal, as on the breakout D41: NOT FITTED. fast-release option (remove the 0R) D42: NOT FITTED. D43: NOT FITTED. D44: NOT FITTED. D45: NOT FITTED. D46: NOT FITTED. D47: NOT FITTED. D48: NOT FITTED. U16: serial mode; internal DC/DC off (DC_ENA low), field side from VBB. Values from Inf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"
- note added: "R118: 22.1k: about 500 kHz scan (datasheet typical) R119: type 1 (eval board RTS = 33 ohm; datasheet: type 2 = 33k, type 3 = 330k). CHECK type 1 value R120: wire-break current, 25-55k range (datasheet curves) R122: RIN, eval board R123: RLED (no LED here; the breakout has them) J10: same pinout as the breakout J1, standard straight-through 40-way ribbon F10: ribbon +24 V: sensor supply and breako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"
- note removed: "D48: NOT FITTED. U16: serial mode; internal DC/DC off (DC_ENA low), field side from VBB. Values from Infineon's ISO1I813T evaluation board. Pinout checked against the datasheet (31 Oct): serial mode 3 (24-bit, CRC) R118: 22.1k: about 500 kHz scan (datasheet typical) R119: type 1 (eval board RTS = 33 ohm; datasheet: type 2 = 33k, type 3 = 330k). CHECK type 1 value R120: wire-break current, 25-55k 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"
- note removed: "U15: pinout checked against DS14170 (31 Oct). Tab = VCC (+24V_FB): copper pour on the field side only C200: bank B bulk J11: 8 A return over 2 contacts: CHECK the plug rating (8 A per contact) D31: flyback at the terminal, as on the breakout D41: NOT FITTED. fast-release option (remove the 0R) D42: NOT FITTED. D43: NOT FITTED. D44: NOT FITTED. D45: NOT FITTED. D46: NOT FITTED. D47: NOT FITTED."
- moved on the sheet: R138, R139, R140, R141, R142, R143
