File: hardware/io_breakout/channels.kicad_sch (KiCad schematic)
At the start: 56 parts

Commit message: One 40-way ribbon for all digital I/O (Gary, 31 Oct)
Main board: J10 becomes a 40-way latched IDC header carrying bank A outputs 1-8 (pins
1-16, each beside its 0 V) and inputs 1-8 (pins 17-32), with 4 x +24 V and 4 x 0 V; J12
and F11 removed, so no ribbon can go into the wrong slot. Breakout rev 0.2: one board,
50 x 80 mm, two-tier 3.81 mm pluggable headers (valves OUT over 0V, inputs IN over +24V,
plus a 0V strip for 3-wire sensors), LEDs on every channel, flyback options on the valves.
Two-tier footprint is a placeholder until the maker's drawing is checked.

Co-Authored-By: Claude Opus 5.5 <noreply@anthropic.com>
Claude-Session: https://claude.ai/code/session_014onnq3eRiDkqdAB6fKiRDW
Parts:
- removed RW1, RW2, RW3, RW4, RW5, RW6, RW7, RW8: DNF, Resistor_SMD:R_0805_2012Metric, symbol Device:R
- added LED11, LED12, LED13, LED14, LED15, LED16, LED17, LED18: yellow, LED_SMD:LED_0805_2012Metric, symbol Device:LED
- added R11, R12, R13, R14, R15, R16, R17, R18: 10k, Resistor_SMD:R_0805_2012Metric, symbol Device:R
Connections:
- net 0V: now also LED11.1 (K), LED12.1 (K), LED13.1 (K), LED14.1 (K), LED15.1 (K), LED16.1 (K), LED17.1 (K), LED18.1 (K)
- net CH1 renamed OUT1
- net CH2 renamed OUT2
- net CH3 renamed OUT3
- net CH4 renamed OUT4
- net CH5 renamed OUT5
- net CH6 renamed OUT6
- net CH7 renamed OUT7
- net CH8 renamed OUT8
- new net IN1: R11.1
- new net IN2: R12.1
- new net IN3: R13.1
- new net IN4: R14.1
- new net IN5: R15.1
- new net IN6: R16.1
- new net IN7: R17.1
- new net IN8: R18.1
- new net LED11_A: LED11.2 (A), R11.2
- new net LED12_A: LED12.2 (A), R12.2
- new net LED13_A: LED13.2 (A), R13.2
- new net LED14_A: LED14.2 (A), R14.2
- new net LED15_A: LED15.2 (A), R15.2
- new net LED16_A: LED16.2 (A), R16.2
- new net LED17_A: LED17.2 (A), R17.2
- new net LED18_A: LED18.2 (A), R18.2
Other:
- note added: "Notes R1: 2.2 mA at 24 V, 48 mW D1: flyback RZ1: fitted = plain diode clamp; remove and fit Z for fast release Z1: NOT FITTED. fast-release option. CHECK Vz + 0.7 V stays below the ISO2H823V2.5's own demagnetisation clamp Z2: NOT FITTED. Z3: NOT FITTED."
- note added: "Z4: NOT FITTED. Z5: NOT FITTED. Z6: NOT FITTED. Z7: NOT FITTED. Z8: NOT FITTED. R11: input LED, 2.2 mA (the input itself draws about 2 mA)"
- note removed: "Notes R1: 2.2 mA at 24 V, 48 mW D1: flyback, OUT build only RZ1: fitted = plain diode clamp; remove and fit Z for fast release Z1: NOT FITTED. fast-release option. CHECK Vz + 0.7 V stays below the ISO2H823V2.5's own demagnetisation clamp RW1: NOT FITTED. normally not fitted: field wire-break needs the bias R at the sensor end; RW here only detects a ribbon break Z2: NOT FITTED. RW2: NOT FITTED. Z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"
- note removed: "RW4: NOT FITTED. Z5: NOT FITTED. RW5: NOT FITTED. Z6: NOT FITTED. RW6: NOT FITTED. Z7: NOT FITTED. RW7: NOT FITTED. Z8: NOT FITTED. RW8: NOT FITTED."
- moved on the sheet: D2, D3, D4, D5, D6, D7, D8, DS2, DS3, DS4, DS5, DS6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
